File: arduino-nano-shield/arduino-nano-shield.kicad_sch (KiCad schematic)
At the start: 16 parts, among them J1 ELRS, J2 M1, J3 M2, J4 LED_D11, J5 LED_D11, J6 SPWR, J7 I2C, J8 SERVO, Q1 BD139, Q2 2N3904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

Commit message: Add V2 board
- jumper for powering second ESC header VCC from main VCC net
- GPS header with D5/D6
- support two servos on servo header
Parts:
- removed J8: SERVO, Connector_PinHeader_2.54mm:PinHeader_1x03_P2.54mm_Vertical, symbol Connector:Conn_01x03_Pin
- added J10: GPS, Connector_PinHeader_2.54mm:PinHeader_1x04_P2.54mm_Vertical, symbol Connector:Conn_01x04_Pin
- added J8: SERVO, Connector_PinHeader_2.54mm:PinHeader_2x03_P2.54mm_Vertical, symbol Connector_Generic:Conn_02x03_Odd_Even
- added J9: JP1, Connector_PinHeader_2.54mm:PinHeader_1x02_P2.54mm_Vertical, symbol Connector:Conn_01x02_Pin
Connections:
- net D10: now also J8.1 (Pin_1), J8.2 (Pin_2)
- net GND: now also J10.1 (Pin_1), J8.5 (Pin_5), J8.6 (Pin_6)
- net VCC: now also J10.4 (Pin_4), J8.3 (Pin_3), J8.4 (Pin_4), J9.1 (Pin_1)
- net at J3.2 (Pin_2), J6.2 (Pin_2), J6.4 (Pin_4)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: now also J9.2 (Pin_2)
- net GTX_D5: now reaches A1.8 (D5)
- net GTX_D5: now also J10.2 (Pin_2)
- net GRX_D6: now reaches A1.9 (D6)
- net GRX_D6: now also J10.3 (Pin_3)

Commit message: Add v2.1 board
- add three pin header as alternative for LED connections (populate
  with angled header) to connect to various multiplexing controllers
- add headers for A20 and A21 as aux connectors
Parts:
- added J11: LED, Connector_PinHeader_2.54mm:PinHeader_1x03_P2.54mm_Vertical, symbol Connector:Conn_01x03_Pin
- added J12: AUX, Connector_PinHeader_2.54mm:PinHeader_1x02_P2.54mm_Vertical, symbol Connector:Conn_01x02_Pin
Connections:
- net at A1.14 (MOSI), R3.2: now also J11.1 (Pin_1)
- net at A1.15 (MISO): now also J11.2 (Pin_2)
- net at A1.16 (SCK), R2.2: now also J11.3 (Pin_3)
- net at A1.20 (A1): now also J12.2 (Pin_2)
- net at A1.21 (A2): now also J12.1 (Pin_1)
Other:
- moved on the sheet: R3
